File: EggPCB/_autosave-EggPCB.kicad_pcb (KiCad board)
At the start: 2 copper layers, 32.6 x 23.2 mm, 11 parts, among them J1 Photocell_1_V+, J2 Photocell_2_V+, J3 Photocell_1_V-, J4 Photocell_2_V-, J5 Conn_01x02_Pin, J6 Conn_01x02_Pin, J7 Photocell_1_V-, J8 GND VIA

Commit message: Nicla to Raspi connection should be working
Parts:
- moved R5 1.50 mm to (110.2, 108.8)
Routing:
- net GND: track 27.0 -> 28.5 mm
- net ADC1: track 19.4 -> 20.3 mm
- net ADC2: track 25.2 -> 24.4 mm
Changed lines of the file:
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@@
 	(footprint "Resistor_SMD:R_0603_1608Metric_Pad0.98x0.95mm_HandSolder"
 		(layer "F.Cu")
-		(at 110.1625 110.25)
+		(at 110.1625 108.75)
 		(descr "Resistor SMD 0603 (1608 Metric), square (rectangular) end terminal, IPC-7351 nominal with elongated pad for handsoldering. (Body size source: IPC-SM-782 page 72, https://www.pcb-3d.com/wordpress/wp-content/uploads/ipc-sm-782a_amendment_1_and_2.pdf), generated with kicad-footprint-generator")
 		(tags "resistor handsolder")
@@
 	)
 	(segment
+		(start 107.95 100.33)
+		(end 107.95 105.35)
+		(width 0.8)
+		(layer "F.Cu")
+		(net 1)
+	)
+	(segment
 		(start 109.25 106.65)
+		(end 109.25 108.75)
+		(width 0.8)
+		(layer "F.Cu")
+		(net 1)
+	)
+	(segment
+		(start 115.57 102.93)
 		(end 115.57 100.33)
 		(width 0.8)
@@
 	)
 	(segment
+		(start 108.1 105.5)
+		(end 113 105.5)
+		(width 0.8)
+		(layer "F.Cu")
+		(net 1)
+	)
+	(segment
+		(start 113 105.5)
+		(end 115.57 102.93)
+		(width 0.8)
+		(layer "F.Cu")
+		(net 1)
+	)
+	(segment
 		(start 107.95 105.35)
-		(end 107.95 100.33)
+		(end 109.25 106.65)
 		(width 0.8)
 		(layer "F.Cu")
@@
 	)
 	(segment
-		(start 109.25 106.65)
-		(end 107.95 105.35)
+		(start 107.95 105.35)
+		(end 108.1 105.5)
 		(width 0.8)
 		(layer "F.Cu")
@@
 	)
 	(segment
-		(start 109.25 110.25)
-		(end 109.25 106.65)
-		(width 0.8)
-		(layer "F.Cu")
-		(net 1)
-	)
-	(segment
-		(start 104.5 112.75)
-		(end 104.5 101.24)
+		(start 105.5 100.42)
+		(end 105.41 100.33)
+		(width 0.8)
+		(layer "F.Cu")
+		(net 2)
+	)
+	(segment
+		(start 105.5 113.75)
+		(end 105.5 100.42)
 		(width 0.8)
 		(layer "F.Cu")
@@
 	)
 	(segment
-		(start 106.75 115)
-		(end 104.5 112.75)
-		(width 0.8)
-		(layer "F.Cu")
-		(net 2)
-	)
-	(segment
 		(start 106.75 120.58)
 		(end 106.68 120.65)
@@
 	)
 	(segment
-		(start 104.5 101.24)
-		(end 105.41 100.33)
+		(start 106.75 115)
+		(end 105.5 113.75)
 		(width 0.8)
 		(layer "F.Cu")
@@
 	)
 	(segment
-		(start 111.075 110.25)
-		(end 111.075 112.5)
-		(width 0.8)
-		(layer "F.Cu")
-		(net 3)
-	)
-	(segment
 		(start 110.49 120.65)
 		(end 110.49 120.51)
 		(width 0.8)
 		(layer "F.Cu")
+		(net 3)
+	)
+	(segment
+		(start 111.075 112.5)
+		(end 111.075 108.75)
+		(width 0.8)
+		(layer "F.Cu")
